File: SheepyPad.kicad_pcb (KiCad board)
At the start: 2 copper layers, 127.6 x 99.7 mm, 60 parts, among them SW1 SW_Push, SW2 Rotary_Encoder_Switch, U1 Sparkfun_Pro_Micro

Commit message: Updates
Parts:
- moved C6 9.92 mm to (71.8, 52.1), turned to 270 degrees
- moved C5 5.50 mm to (120.3, 64.8), turned to 0 degrees
- moved C3 5.08 mm to (168.9, 121.9), turned to 180 degrees
- moved C4 5.00 mm to (168.8, 64.8), turned to 180 degrees
- moved C1 4.95 mm to (78.2, 88.3), turned to 0 degrees
- moved D22 1.42 mm to (66.0, 54.6), turned to 180 degrees
- moved C2 0.08 mm to (120.7, 121.9)
Connections:
- U1 pad 1: /ENC_B -> /ENC_A
- U1 pad 2: /ENC_A -> /ENC_B
Routing:
- net +5V: track 18.2 -> 324.3 mm, vias 6 -> 1
- net /RESET: track 33.5 -> 51.7 mm
- net /ENC_A: track 16.6 -> 22.5 mm
- net /GLOW_LED: track 19.8 -> 22.9 mm
- net /ENC_B: track 14.2 -> 11.6 mm
- net Net-(D24-Pad2): track 51.1 -> 49.7 mm
- net Net-(D23-Pad2): track 61.3 -> 62.6 mm
- net /ROW_5: track 145.9 -> 145.0 mm
- net /COL_ENC_1: track 22.6 -> 23.5 mm
- net Net-(D22-Pad2): track 70.3 -> 69.6 mm
- added copper zone on F.Cu, net GND
- removed copper zone on F.Cu, net +5V
