File: SheepyPad.kicad_pcb (KiCad board)
At the start: 2 copper layers, 127.6 x 99.7 mm, 60 parts, among them SW1 SW_Push, SW2 Rotary_Encoder_Switch, U1 Sparkfun_Pro_Micro

Commit message: Update fabrication
Parts:
- removed the G*** at (95.9, 72.4)
- added G***: LOGO, Logos:Sleepy, F.Cu at (95.6, 72.3)
