File: Hardware/SheepyPad.sch (KiCad schematic (older format))
At the start: 58 parts, among them SW1 SW_Push, SW2 Rotary_Encoder_Switch, U1 Sparkfun_Pro_Micro

Commit message: Fixed Diode orientation for encoder SW
Connections:
- net COL_ENC_1: now also D21.2 (A); no longer D21.1 (K)
- net at SW2.S1: now also D21.1 (K); no longer D21.2 (A)
Changed lines of the file:
@@
 Text Label 8700 5750 0    50   ~ 0
 COL_ENC_1
-Wire Wire Line
-	8000 5750 8100 5750
 $Comp
 L Device:D_Small D21
@@
 F 3 "~" V 8200 5750 50  0001 C CNN
 	1    8200 5750
-	-1   0    0    1
-$EndComp
-Wire Wire Line
-	8300 5750 8700 5750
+	1    0    0    -1
+$EndComp
 Text Notes 7150 5250 0    100  ~ 0
 Rotary Encoder
@@
 	2700 4250 2300 4250
 Connection ~ 2300 4250
+Wire Wire Line
+	8300 5750 8700 5750
+Wire Wire Line
+	8100 5750 8000 5750
 $EndSCHEMATC
