File: Hardware/v2/SheepyPad.sch (KiCad schematic (older format))
At the start: 58 parts, among them SW1 SW_Push, SW2 Rotary_Encoder_Switch, U1 Sparkfun_Pro_Micro

Commit message: Remove of redundant lib
Parts:
- MX1, MX10, MX11, MX12, MX13, MX14, MX15, MX16, MX17, MX18, MX19, MX2, MX20, MX3, MX4, MX5, MX6, MX7, MX8, MX9: footprint MX_Only:MXOnly-1U-NoLED -> Keyswitches:Kailh_socket_MX_optional_reversible_FLIP
Changed lines of the file:
@@
 F 0 "MX2" H 7233 2523 60  0000 C CNN
 F 1 "MX-NoLED" H 7233 2449 20  0000 C CNN
-F 2 "MX_Only:MXOnly-1U-NoLED" H 6575 2275 60  0001 C CNN
+F 2 "Keyswitches:Kailh_socket_MX_optional_reversible_FLIP" H 6575 2275 60  0001 C CNN
 F 3 "" H 6575 2275 60  0001 C CNN
 	1    7200 2300
@@
 F 0 "MX7" H 7783 2523 60  0000 C CNN
 F 1 "MX-NoLED" H 7783 2449 20  0000 C CNN
-F 2 "MX_Only:MXOnly-1U-NoLED" H 7125 2275 60  0001 C CNN
+F 2 "Keyswitches:Kailh_socket_MX_optional_reversible_FLIP" H 7125 2275 60  0001 C CNN
 F 3 "" H 7125 2275 60  0001 C CNN
 	1    7750 2300
@@
 F 0 "MX12" H 8333 2523 60  0000 C CNN
 F 1 "MX-NoLED" H 8333 2449 20  0000 C CNN
-F 2 "MX_Only:MXOnly-1U-NoLED" H 7675 2275 60  0001 C CNN
+F 2 "Keyswitches:Kailh_socket_MX_optional_reversible_FLIP" H 7675 2275 60  0001 C CNN
 F 3 "" H 7675 2275 60  0001 C CNN
 	1    8300 2300
@@
 F 0 "MX3" H 7233 3173 60  0000 C CNN
 F 1 "MX-NoLED" H 7233 3099 20  0000 C CNN
-F 2 "MX_Only:MXOnly-1U-NoLED" H 6575 2925 60  0001 C CNN
+F 2 "Keyswitches:Kailh_socket_MX_optional_reversible_FLIP" H 6575 2925 60  0001 C CNN
 F 3 "" H 6575 2925 60  0001 C CNN
 	1    7200 2950
@@
 F 0 "MX8" H 7783 3173 60  0000 C CNN
 F 1 "MX-NoLED" H 7783 3099 20  0000 C CNN
-F 2 "MX_Only:MXOnly-1U-NoLED" H 7125 2925 60  0001 C CNN
+F 2 "Keyswitches:Kailh_socket_MX_optional_reversible_FLIP" H 7125 2925 60  0001 C CNN
 F 3 "" H 7125 2925 60  0001 C CNN
 	1    7750 2950
@@
 F 0 "MX13" H 8333 3173 60  0000 C CNN
 F 1 "MX-NoLED" H 8333 3099 20  0000 C CNN
-F 2 "MX_Only:MXOnly-1U-NoLED" H 7675 2925 60  0001 C CNN
+F 2 "Keyswitches:Kailh_socket_MX_optional_reversible_FLIP" H 7675 2925 60  0001 C CNN
 F 3 "" H 7675 2925 60  0001 C CNN
 	1    8300 2950
@@
 F 0 "MX15" H 8333 4473 60  0000 C CNN
 F 1 "MX-NoLED" H 8333 4399 20  0000 C CNN
-F 2 "MX_Only:MXOnly-1U-NoLED" H 7675 4225 60  0001 C CNN
+F 2 "Keyswitches:Kailh_socket_MX_optional_reversible_FLIP" H 7675 4225 60  0001 C CNN
 F 3 "" H 7675 4225 60  0001 C CNN
 	1    8300 4250
@@
 F 0 "MX10" H 7783 4473 60  0000 C CNN
 F 1 "MX-NoLED" H 7783 4399 20  0000 C CNN
-F 2 "MX_Only:MXOnly-1U-NoLED" H 7125 4225 60  0001 C CNN
+F 2 "Keyswitches:Kailh_socket_MX_optional_reversible_FLIP" H 7125 4225 60  0001 C CNN
 F 3 "" H 7125 4225 60  0001 C CNN
 	1    7750 4250
@@
 F 0 "MX5" H 7233 4473 60  0000 C CNN
 F 1 "MX-NoLED" H 7233 4399 20  0000 C CNN
-F 2 "MX_Only:MXOnly-1U-NoLED" H 6575 4225 60  0001 C CNN
+F 2 "Keyswitches:Kailh_socket_MX_optional_reversible_FLIP" H 6575 4225 60  0001 C CNN
 F 3 "" H 6575 4225 60  0001 C CNN
 	1    7200 4250
@@
 F 0 "MX14" H 8333 3823 60  0000 C CNN
 F 1 "MX-NoLED" H 8333 3749 20  0000 C CNN
-F 2 "MX_Only:MXOnly-1U-NoLED" H 7675 3575 60  0001 C CNN
+F 2 "Keyswitches:Kailh_socket_MX_optional_reversible_FLIP" H 7675 3575 60  0001 C CNN
 F 3 "" H 7675 3575 60  0001 C CNN
 	1    8300 3600
@@
 F 0 "MX9" H 7783 3823 60  0000 C CNN
 F 1 "MX-NoLED" H 7783 3749 20  0000 C CNN
-F 2 "MX_Only:MXOnly-1U-NoLED" H 7125 3575 60  0001 C CNN
+F 2 "Keyswitches:Kailh_socket_MX_optional_reversible_FLIP" H 7125 3575 60  0001 C CNN
 F 3 "" H 7125 3575 60  0001 C CNN
 	1    7750 3600
@@
 F 0 "MX4" H 7233 3823 60  0000 C CNN
 F 1 "MX-NoLED" H 7233 3749 20  0000 C CNN
-F 2 "MX_Only:MXOnly-1U-NoLED" H 6575 3575 60  0001 C CNN
+F 2 "Keyswitches:Kailh_socket_MX_optional_reversible_FLIP" H 6575 3575 60  0001 C CNN
 F 3 "" H 6575 3575 60  0001 C CNN
 	1    7200 3600
@@
 F 0 "MX6" H 7783 1873 60  0000 C CNN
 F 1 "MX-NoLED" H 7783 1799 20  0000 C CNN
-F 2 "MX_Only:MXOnly-1U-NoLED" H 7125 1625 60  0001 C CNN
+F 2 "Keyswitches:Kailh_socket_MX_optional_reversible_FLIP" H 7125 1625 60  0001 C CNN
 F 3 "" H 7125 1625 60  0001 C CNN
 	1    7750 1650
@@
 F 0 "MX11" H 8333 1873 60  0000 C CNN
 F 1 "MX-NoLED" H 8333 1799 20  0000 C CNN
-F 2 "MX_Only:MXOnly-1U-NoLED" H 7675 1625 60  0001 C CNN
+F 2 "Keyswitches:Kailh_socket_MX_optional_reversible_FLIP" H 7675 1625 60  0001 C CNN
 F 3 "" H 7675 1625 60  0001 C CNN
 	1    8300 1650
@@
 F 0 "MX17" H 8883 2523 60  0000 C CNN
 F 1 "MX-NoLED" H 8883 2449 20  0000 C CNN
-F 2 "MX_Only:MXOnly-1U-NoLED" H 8225 2275 60  0001 C CNN
+F 2 "Keyswitches:Kailh_socket_MX_optional_reversible_FLIP" H 8225 2275 60  0001 C CNN
 F 3 "" H 8225 2275 60  0001 C CNN
 	1    8850 2300
@@
 F 0 "MX16" H 8883 1873 60  0000 C CNN
 F 1 "MX-NoLED" H 8883 1799 20  0000 C CNN
-F 2 "MX_Only:MXOnly-1U-NoLED" H 8225 1625 60  0001 C CNN
+F 2 "Keyswitches:Kailh_socket_MX_optional_reversible_FLIP" H 8225 1625 60  0001 C CNN
 F 3 "" H 8225 1625 60  0001 C CNN
 	1    8850 1650
@@
 F 0 "MX1" H 7233 1873 60  0000 C CNN
 F 1 "MX-NoLED" H 7233 1799 20  0000 C CNN
-F 2 "MX_Only:MXOnly-1U-NoLED" H 6575 1625 60  0001 C CNN
+F 2 "Keyswitches:Kailh_socket_MX_optional_reversible_FLIP" H 6575 1625 60  0001 C CNN
 F 3 "" H 6575 1625 60  0001 C CNN
 	1    7200 1650
@@
 F 0 "MX18" H 8883 3173 60  0000 C CNN
 F 1 "MX-NoLED" H 8883 3099 20  0000 C CNN
-F 2 "MX_Only:MXOnly-1U-NoLED" H 8225 2925 60  0001 C CNN
+F 2 "Keyswitches:Kailh_socket_MX_optional_reversible_FLIP" H 8225 2925 60  0001 C CNN
 F 3 "" H 8225 2925 60  0001 C CNN
 	1    8850 2950
@@
 F 0 "MX19" H 8883 3823 60  0000 C CNN
 F 1 "MX-NoLED" H 8883 3749 20  0000 C CNN
-F 2 "MX_Only:MXOnly-1U-NoLED" H 8225 3575 60  0001 C CNN
+F 2 "Keyswitches:Kailh_socket_MX_optional_reversible_FLIP" H 8225 3575 60  0001 C CNN
 F 3 "" H 8225 3575 60  0001 C CNN
 	1    8850 3600
@@
 F 0 "MX20" H 8883 4473 60  0000 C CNN
 F 1 "MX-NoLED" H 8883 4399 20  0000 C CNN
-F 2 "MX_Only:MXOnly-1U-NoLED" H 8225 4225 60  0001 C CNN
+F 2 "Keyswitches:Kailh_socket_MX_optional_reversible_FLIP" H 8225 4225 60  0001 C CNN
 F 3 "" H 8225 4225 60  0001 C CNN
 	1    8850 4250

Commit message: WIP v2
Parts:
- D1, D10, D11, D12, D13, D14, D15, D16, D17, D18, D19, D2, D20, D21, D3, D4, D5, D6, D7, D8, D9: footprint Diode_THT:D_DO-35_SOD27_P10.16mm_Horizontal -> Random-keyboard-parts:Diode_SMD_THT_DUAL
Changed lines of the file:
@@
 F 0 "D10" V 7546 4430 50  0000 R CNN
 F 1 "D_Small" V 7455 4430 50  0000 R CNN
-F 2 "Diode_THT:D_DO-35_SOD27_P10.16mm_Horizontal" V 7500 4500 50  0001 C CNN
+F 2 "Random-keyboard-parts:Diode_SMD_THT_DUAL" V 7500 4500 50  0001 C CNN
 F 3 "~" V 7500 4500 50  0001 C CNN
 	1    7500 4500
@@
 F 0 "D15" V 8096 4430 50  0000 R CNN
 F 1 "D_Small" V 8005 4430 50  0000 R CNN
-F 2 "Diode_THT:D_DO-35_SOD27_P10.16mm_Horizontal" V 8050 4500 50  0001 C CNN
+F 2 "Random-keyboard-parts:Diode_SMD_THT_DUAL" V 8050 4500 50  0001 C CNN
 F 3 "~" V 8050 4500 50  0001 C CNN
 	1    8050 4500
@@
 F 0 "D5" V 6996 4430 50  0000 R CNN
 F 1 "D_Small" V 6905 4430 50  0000 R CNN
-F 2 "Diode_THT:D_DO-35_SOD27_P10.16mm_Horizontal" V 6950 4500 50  0001 C CNN
+F 2 "Random-keyboard-parts:Diode_SMD_THT_DUAL" V 6950 4500 50  0001 C CNN
 F 3 "~" V 6950 4500 50  0001 C CNN
 	1    6950 4500
@@
 F 0 "D14" V 8096 3780 50  0000 R CNN
 F 1 "D_Small" V 8005 3780 50  0000 R CNN
-F 2 "Diode_THT:D_DO-35_SOD27_P10.16mm_Horizontal" V 8050 3850 50  0001 C CNN
+F 2 "Random-keyboard-parts:Diode_SMD_THT_DUAL" V 8050 3850 50  0001 C CNN
 F 3 "~" V 8050 3850 50  0001 C CNN
 	1    8050 3850
@@
 F 0 "D9" V 7546 3780 50  0000 R CNN
 F 1 "D_Small" V 7455 3780 50  0000 R CNN
-F 2 "Diode_THT:D_DO-35_SOD27_P10.16mm_Horizontal" V 7500 3850 50  0001 C CNN
+F 2 "Random-keyboard-parts:Diode_SMD_THT_DUAL" V 7500 3850 50  0001 C CNN
 F 3 "~" V 7500 3850 50  0001 C CNN
 	1    7500 3850
@@
 F 0 "D4" V 6996 3780 50  0000 R CNN
 F 1 "D_Small" V 6905 3780 50  0000 R CNN
-F 2 "Diode_THT:D_DO-35_SOD27_P10.16mm_Horizontal" V 6950 3850 50  0001 C CNN
+F 2 "Random-keyboard-parts:Diode_SMD_THT_DUAL" V 6950 3850 50  0001 C CNN
 F 3 "~" V 6950 3850 50  0001 C CNN
 	1    6950 3850
@@
 F 0 "D3" V 6996 3130 50  0000 R CNN
 F 1 "D_Small" V 6905 3130 50  0000 R CNN
-F 2 "Diode_THT:D_DO-35_SOD27_P10.16mm_Horizontal" V 6950 3200 50  0001 C CNN
+F 2 "Random-keyboard-parts:Diode_SMD_THT_DUAL" V 6950 3200 50  0001 C CNN
 F 3 "~" V 6950 3200 50  0001 C CNN
 	1    6950 3200
@@
 F 0 "D8" V 7546 3130 50  0000 R CNN
 F 1 "D_Small" V 7455 3130 50  0000 R CNN
-F 2 "Diode_THT:D_DO-35_SOD27_P10.16mm_Horizontal" V 7500 3200 50  0001 C CNN
+F 2 "Random-keyboard-parts:Diode_SMD_THT_DUAL" V 7500 3200 50  0001 C CNN
 F 3 "~" V 7500 3200 50  0001 C CNN
 	1    7500 3200
@@
 F 0 "D13" V 8096 3130 50  0000 R CNN
 F 1 "D_Small" V 8005 3130 50  0000 R CNN
-F 2 "Diode_THT:D_DO-35_SOD27_P10.16mm_Horizontal" V 8050 3200 50  0001 C CNN
+F 2 "Random-keyboard-parts:Diode_SMD_THT_DUAL" V 8050 3200 50  0001 C CNN
 F 3 "~" V 8050 3200 50  0001 C CNN
 	1    8050 3200
@@
 F 0 "D12" V 8096 2480 50  0000 R CNN
 F 1 "D_Small" V 8005 2480 50  0000 R CNN
-F 2 "Diode_THT:D_DO-35_SOD27_P10.16mm_Horizontal" V 8050 2550 50  0001 C CNN
+F 2 "Random-keyboard-parts:Diode_SMD_THT_DUAL" V 8050 2550 50  0001 C CNN
 F 3 "~" V 8050 2550 50  0001 C CNN
 	1    8050 2550
@@
 F 0 "D7" V 7546 2480 50  0000 R CNN
 F 1 "D_Small" V 7455 2480 50  0000 R CNN
-F 2 "Diode_THT:D_DO-35_SOD27_P10.16mm_Horizontal" V 7500 2550 50  0001 C CNN
+F 2 "Random-keyboard-parts:Diode_SMD_THT_DUAL" V 7500 2550 50  0001 C CNN
 F 3 "~" V 7500 2550 50  0001 C CNN
 	1    7500 2550
@@
 F 0 "D2" V 6996 2480 50  0000 R CNN
 F 1 "D_Small" V 6905 2480 50  0000 R CNN
-F 2 "Diode_THT:D_DO-35_SOD27_P10.16mm_Horizontal" V 6950 2550 50  0001 C CNN
+F 2 "Random-keyboard-parts:Diode_SMD_THT_DUAL" V 6950 2550 50  0001 C CNN
 F 3 "~" V 6950 2550 50  0001 C CNN
 	1    6950 2550
@@
 F 0 "D1" V 6996 1830 50  0000 R CNN
 F 1 "D_Small" V 6905 1830 50  0000 R CNN
-F 2 "Diode_THT:D_DO-35_SOD27_P10.16mm_Horizontal" V 6950 1900 50  0001 C CNN
+F 2 "Random-keyboard-parts:Diode_SMD_THT_DUAL" V 6950 1900 50  0001 C CNN
 F 3 "~" V 6950 1900 50  0001 C CNN
 	1    6950 1900
@@
 F 0 "D6" V 7546 1830 50  0000 R CNN
 F 1 "D_Small" V 7455 1830 50  0000 R CNN
-F 2 "Diode_THT:D_DO-35_SOD27_P10.16mm_Horizontal" V 7500 1900 50  0001 C CNN
+F 2 "Random-keyboard-parts:Diode_SMD_THT_DUAL" V 7500 1900 50  0001 C CNN
 F 3 "~" V 7500 1900 50  0001 C CNN
 	1    7500 1900
@@
 F 0 "D11" V 8096 1830 50  0000 R CNN
 F 1 "D_Small" V 8005 1830 50  0000 R CNN
-F 2 "Diode_THT:D_DO-35_SOD27_P10.16mm_Horizontal" V 8050 1900 50  0001 C CNN
+F 2 "Random-keyboard-parts:Diode_SMD_THT_DUAL" V 8050 1900 50  0001 C CNN
 F 3 "~" V 8050 1900 50  0001 C CNN
 	1    8050 1900
@@
 F 0 "D16" V 8646 1830 50  0000 R CNN
 F 1 "D_Small" V 8555 1830 50  0000 R CNN
-F 2 "Diode_THT:D_DO-35_SOD27_P10.16mm_Horizontal" V 8600 1900 50  0001 C CNN
+F 2 "Random-keyboard-parts:Diode_SMD_THT_DUAL" V 8600 1900 50  0001 C CNN
 F 3 "~" V 8600 1900 50  0001 C CNN
 	1    8600 1900
@@
 F 0 "D17" V 8646 2480 50  0000 R CNN
 F 1 "D_Small" V 8555 2480 50  0000 R CNN
-F 2 "Diode_THT:D_DO-35_SOD27_P10.16mm_Horizontal" V 8600 2550 50  0001 C CNN
+F 2 "Random-keyboard-parts:Diode_SMD_THT_DUAL" V 8600 2550 50  0001 C CNN
 F 3 "~" V 8600 2550 50  0001 C CNN
 	1    8600 2550
@@
 F 0 "D18" V 8646 3130 50  0000 R CNN
 F 1 "D_Small" V 8555 3130 50  0000 R CNN
-F 2 "Diode_THT:D_DO-35_SOD27_P10.16mm_Horizontal" V 8600 3200 50  0001 C CNN
+F 2 "Random-keyboard-parts:Diode_SMD_THT_DUAL" V 8600 3200 50  0001 C CNN
 F 3 "~" V 8600 3200 50  0001 C CNN
 	1    8600 3200
@@
 F 0 "D19" V 8646 3780 50  0000 R CNN
 F 1 "D_Small" V 8555 3780 50  0000 R CNN
-F 2 "Diode_THT:D_DO-35_SOD27_P10.16mm_Horizontal" V 8600 3850 50  0001 C CNN
+F 2 "Random-keyboard-parts:Diode_SMD_THT_DUAL" V 8600 3850 50  0001 C CNN
 F 3 "~" V 8600 3850 50  0001 C CNN
 	1    8600 3850
@@
 F 0 "D20" V 8646 4430 50  0000 R CNN
 F 1 "D_Small" V 8555 4430 50  0000 R CNN
-F 2 "Diode_THT:D_DO-35_SOD27_P10.16mm_Horizontal" V 8600 4500 50  0001 C CNN
+F 2 "Random-keyboard-parts:Diode_SMD_THT_DUAL" V 8600 4500 50  0001 C CNN
 F 3 "~" V 8600 4500 50  0001 C CNN
 	1    8600 4500
@@
 F 0 "D21" H 8246 5680 50  0000 R CNN
 F 1 "D_Small" H 8155 5680 50  0000 R CNN
-F 2 "Diode_THT:D_DO-35_SOD27_P10.16mm_Horizontal" V 8200 5750 50  0001 C CNN
+F 2 "Random-keyboard-parts:Diode_SMD_THT_DUAL" V 8200 5750 50  0001 C CNN
 F 3 "~" V 8200 5750 50  0001 C CNN
 	1    8200 5750

Commit message: Update
Parts:
- removed R1: 10K, Resistor_THT:R_Axial_DIN0207_L6.3mm_D2.5mm_P10.16mm_Horizontal, symbol Device:R
Connections:
- net ROW_1: now also SW2.S2
- net COL_ENC_1 renamed COL_0
- net ROW_ENC_1: no longer names the net of U1.8 (PC6)
- net ROW_ENC_1: no longer SW2.S2
Changed lines of the file:
@@
 	7200 5850 7400 5850
 Text Label 8700 5950 0    50   ~ 0
-ROW_ENC_1
+ROW_1
 $Comp
 L power:GND #PWR0101
@@
 Text Notes 6450 1000 0    100  ~ 0
 Switch Matrix
-Text Label 5900 6100 0    50   ~ 0
+Text Label 5750 6100 0    50   ~ 0
 RESET
-Wire Wire Line
-	5800 5700 5800 5600
-Wire Wire Line
-	5800 6100 5900 6100
-Connection ~ 5800 6100
-Wire Wire Line
-	5800 6000 5800 6100
-Wire Wire Line
-	5500 6100 5800 6100
-Text Notes 4950 5300 0    100  ~ 0
+Text Notes 4900 5600 0    100  ~ 0
 Reset Switch
 Wire Wire Line
@@
 	1    0    0    -1
 $EndComp
-$Comp
-L Device:R R1
-U 1 1 613FAC92
-P 5800 5850
-F 0 "R1" V 5593 5850 50  0000 C CNN
-F 1 "10K" V 5684 5850 50  0000 C CNN
-F 2 "Resistor_THT:R_Axial_DIN0207_L6.3mm_D2.5mm_P10.16mm_Horizontal" V 5730 5850 50  0001 C CNN
-F 3 "~" H 5800 5850 50  0001 C CNN
-	1    5800 5850
-	1    0    0    -1
-$EndComp
-$Comp
-L power:+5V #PWR0104
-U 1 1 613FA72E
-P 5800 5600
-F 0 "#PWR0104" H 5800 5450 50  0001 C CNN
-F 1 "+5V" H 5815 5773 50  0000 C CNN
-F 2 "" H 5800 5600 50  0001 C CNN
-F 3 "" H 5800 5600 50  0001 C CNN
-	1    5800 5600
-	1    0    0    -1
-$EndComp
 Wire Wire Line
 	7400 5750 6700 5750
@@
 ENC_A
 Text Label 8700 5750 0    50   ~ 0
-COL_ENC_1
+COL_0
 $Comp
 L Device:D_Small D21
@@
 Text Notes 7150 5250 0    100  ~ 0
 Rotary Encoder
-Text Label 2100 5500 0    50   ~ 0
-ROW_ENC_1
 Text Label 2100 5400 0    50   ~ 0
-COL_ENC_1
+COL_0
 Wire Wire Line
 	2100 5500 2550 5500
@@
 Wire Wire Line
 	8100 5750 8000 5750
+Wire Wire Line
+	5500 6100 5750 6100
 $EndSCHEMATC

Commit message: Update v2
Connections:
- net COL_0: now also U1.13 (PB6); no longer U1.7 (PD4)
- net COL_1: now also U1.14 (PB2); no longer U1.16 (PB1)
- net COL_3: now also U1.16 (PB1); no longer U1.14 (PB2)
- net COL_4: now also U1.17 (PF7); no longer U1.13 (PB6)
- net ENC_A: now also U1.19 (PF5); no longer U1.1 (PD3)
- net ENC_B: now also U1.20 (PF4); no longer U1.2 (PD2)
- net GLOW_LED: now also U1.7 (PD4); no longer U1.18 (PF6)
- net ROW_1: now also D12.1 (K), D17.1 (K), D2.1 (K), D7.1 (K), U1.11 (PB4); no longer D1.1 (K), D11.1 (K), D16.1 (K), D6.1 (K), SW2.S2, U1.17 (PF7)
- net ROW_2: now also D13.1 (K), D18.1 (K), D3.1 (K), D8.1 (K), U1.10 (PE6); no longer D12.1 (K), D17.1 (K), D2.1 (K), D7.1 (K), U1.12 (PB5)
- net ROW_3: now also D14.1 (K), D19.1 (K), D4.1 (K), D9.1 (K), U1.9 (PD7); no longer D13.1 (K), D18.1 (K), D3.1 (K), D8.1 (K), U1.11 (PB4)
- net ROW_4: now also D10.1 (K), D15.1 (K), D20.1 (K), D5.1 (K), U1.8 (PC6); no longer D14.1 (K), D19.1 (K), D4.1 (K), D9.1 (K), U1.10 (PE6)
- removed net ROW_5: D10.1 (K), D15.1 (K), D20.1 (K), D5.1 (K), U1.9 (PD7)
- new net DATA: U1.2 (PD2)
- new net ROW_0: D1.1 (K), D11.1 (K), D16.1 (K), D6.1 (K), SW2.S2, U1.12 (PB5)
- no-connect marks 0 -> 1
Changed lines of the file:
@@
 	7200 5850 7400 5850
 Text Label 8700 5950 0    50   ~ 0
-ROW_1
+ROW_0
 $Comp
 L power:GND #PWR0101
@@
 	9000 3550 9000 4200
 Wire Wire Line
-	2550 5900 2150 5900
+	2550 5700 2150 5700
+Wire Wire Line
+	2550 5600 2150 5600
+Wire Wire Line
+	2550 5500 2150 5500
 Wire Wire Line
 	2550 5800 2150 5800
-Wire Wire Line
-	2550 5700 2150 5700
-Wire Wire Line
-	2550 5600 2150 5600
 Text Label 6450 2000 0    50   ~ 0
+ROW_0
+Text Label 6450 2650 0    50   ~ 0
 ROW_1
-Text Label 6450 2650 0    50   ~ 0
+Text Label 6450 3300 0    50   ~ 0
 ROW_2
-Text Label 6450 3300 0    50   ~ 0
+Text Label 6450 3950 0    50   ~ 0
 ROW_3
-Text Label 6450 3950 0    50   ~ 0
+Text Label 6450 4600 0    50   ~ 0
 ROW_4
-Text Label 6450 4600 0    50   ~ 0
-ROW_5
 Text Label 7350 1200 0    50   ~ 0
 COL_1
@@
 Text Label 9000 1200 0    50   ~ 0
 COL_4
-Text Label 4150 5500 2    50   ~ 0
+Text Label 2150 5800 0    50   ~ 0
 ROW_1
-Text Label 2150 5900 0    50   ~ 0
+Text Label 2150 5700 0    50   ~ 0
 ROW_2
-Text Label 2150 5800 0    50   ~ 0
+Text Label 2150 5600 0    50   ~ 0
 ROW_3
-Text Label 2150 5700 0    50   ~ 0
+Text Label 2150 5500 0    50   ~ 0
 ROW_4
 Text Notes 6450 1000 0    100  ~ 0
@@
 	2550 5300 2150 5300
 Text Label 2150 4900 0    50   ~ 0
-ENC_B
+DATA
 Wire Wire Line
 	8000 5950 8700 5950
 Wire Wire Line
-	3750 5900 4150 5900
-Wire Wire Line
-	3750 5800 4150 5800
-Text Label 2150 5600 0    50   ~ 0
-ROW_5
-Text Label 2150 4800 0    50   ~ 0
+	3750 5500 4150 5500
+Wire Wire Line
+	3750 5600 4150 5600
+Text Label 2150 5900 0    50   ~ 0
+ROW_0
+Text Label 4150 5300 2    50   ~ 0
 ENC_A
 Text Label 8700 5750 0    50   ~ 0
@@
 Text Notes 7150 5250 0    100  ~ 0
 Rotary Encoder
-Text Label 2100 5400 0    50   ~ 0
+Text Label 4150 5900 2    50   ~ 0
 COL_0
-Wire Wire Line
-	2100 5500 2550 5500
 $Comp
 L SSD1306-128x64_OLED:SSD1306 Brd1
@@
 Wire Wire Line
 	4200 3100 4750 3100
-Wire Wire Line
-	3750 5400 4400 5400
-Text Label 4400 5400 2    50   ~ 0
+Text Label 2100 5400 0    50   ~ 0
 GLOW_LED
 Wire Wire Line
@@
 OLED Screen
 Wire Wire Line
-	3750 5500 4150 5500
-Wire Wire Line
-	3750 5600 4150 5600
+	3750 5900 4150 5900
+Wire Wire Line
+	3750 5800 4150 5800
 Wire Wire Line
 	3750 5700 4150 5700
-Text Label 4150 5600 2    50   ~ 0
+Text Label 4150 5800 2    50   ~ 0
 COL_1
 Text Label 4150 5700 2    50   ~ 0
 COL_2
-Text Label 4150 5800 2    50   ~ 0
+Text Label 4150 5600 2    50   ~ 0
 COL_3
-Text Label 4150 5900 2    50   ~ 0
+Text Label 4150 5500 2    50   ~ 0
 COL_4
 Wire Wire Line
-	2550 4800 2150 4800
+	3750 5300 4150 5300
 Wire Wire Line
 	2550 4900 2150 4900
@@
 Wire Wire Line
 	5500 6100 5750 6100
+Wire Wire Line
+	2150 5900 2550 5900
+Text Label 4150 5200 2    50   ~ 0
+ENC_B
+Wire Wire Line
+	3750 5200 4150 5200
+NoConn ~ 3750 4800
 $EndSCHEMATC

Commit message: WIP
Parts:
- U1: footprint Arduino:Sparkfun_Pro_Micro -> Arduino:Sparkfun_Pro_Micro_reversible
Changed lines of the file:
@@
 F 0 "U1" H 3150 6289 60  0000 C CNN
 F 1 "Sparkfun_Pro_Micro" H 3150 6183 60  0000 C CNN
-F 2 "Arduino:Sparkfun_Pro_Micro" H 3150 4750 60  0001 C CNN
+F 2 "Arduino:Sparkfun_Pro_Micro_reversible" H 3150 4750 60  0001 C CNN
 F 3 "https://www.sparkfun.com/products/12640" H 3250 4350 60  0001 C CNN
 	1    3150 5400
