File: Hardware/v2/SheepyPad.sch (KiCad schematic (older format))
At the start: 57 parts, among them SW1 SW_Push, SW2 Rotary_Encoder_Switch, U1 Sparkfun_Pro_Micro

Commit message: WIP v2
Parts:
- added J1: AudioJack4, Random-keyboard-parts:PJ-3200B-4A, symbol Connector:AudioJack4
- added JP1: Serial/SCL Jumper, Jumper:SolderJumper-3_P1.3mm_Open_Pad1.0x1.5mm, symbol Jumper:Jumper_3_Open
- added JP2: SDA Jumper, Jumper:SolderJumper-2_P1.3mm_Open_Pad1.0x1.5mm, symbol Device:Jumper
- U1: symbol Arduino:Sparkfun_Pro_Micro -> SheepyPad-rescue:Sparkfun_Pro_Micro-Arduino
Connections:
- net DATA: now also JP1.1 (A)
- net GND: now also J1.T
- net SCL: now also JP1.3 (B)
- net SDA: now also JP2.1
- net +5V renamed VCC
- net VCC: now also J1.S
- new net: J1.R1, JP1.2 (C)
- new net: J1.R2, JP2.2
- no-connect marks 1 -> 4
Changed lines of the file:
@@
 $EndDescr
 $Comp
-L Arduino:Sparkfun_Pro_Micro U1
+L SheepyPad-rescue:Sparkfun_Pro_Micro-Arduino U1
 U 1 1 613F5C32
 P 3150 5400
@@
 L power:GND #PWR0101
 U 1 1 61437620
-P 2550 5000
-F 0 "#PWR0101" H 2550 4750 50  0001 C CNN
-F 1 "GND" V 2555 4872 50  0000 R CNN
-F 2 "" H 2550 5000 50  0001 C CNN
-F 3 "" H 2550 5000 50  0001 C CNN
-	1    2550 5000
-	0    1    1    0
-$EndComp
-$Comp
-L power:GND #PWR0102
-U 1 1 61437D92
-P 2550 5100
-F 0 "#PWR0102" H 2550 4850 50  0001 C CNN
-F 1 "GND" V 2555 4972 50  0000 R CNN
-F 2 "" H 2550 5100 50  0001 C CNN
-F 3 "" H 2550 5100 50  0001 C CNN
-	1    2550 5100
-	0    1    1    0
+P 1950 5100
+F 0 "#PWR0101" H 1950 4850 50  0001 C CNN
+F 1 "GND" H 1955 4972 50  0000 R CNN
+F 2 "" H 1950 5100 50  0001 C CNN
+F 3 "" H 1950 5100 50  0001 C CNN
+	1    1950 5100
+	1    0    0    -1
 $EndComp
 $Comp
@@
 	1    3750 4900
 	0    -1   -1   0
-$EndComp
-$Comp
-L power:+5V #PWR0113
-U 1 1 61439013
-P 3750 5100
-F 0 "#PWR0113" H 3750 4950 50  0001 C CNN
-F 1 "+5V" V 3765 5228 50  0000 L CNN
-F 2 "" H 3750 5100 50  0001 C CNN
-F 3 "" H 3750 5100 50  0001 C CNN
-	1    3750 5100
-	0    1    1    0
 $EndComp
 Wire Wire Line
@@
 	0    -1   -1   0
 $EndComp
-$Comp
-L power:+5V #PWR0107
-U 1 1 6156C119
-P 5400 4500
-F 0 "#PWR0107" H 5400 4350 50  0001 C CNN
-F 1 "+5V" V 5415 4628 50  0000 L CNN
-F 2 "" H 5400 4500 50  0001 C CNN
-F 3 "" H 5400 4500 50  0001 C CNN
-	1    5400 4500
-	0    1    1    0
-$EndComp
 Wire Wire Line
 	5400 4700 5800 4700
@@
 Text Label 2000 1950 0    50   ~ 0
 GLOW_LED
-$Comp
-L power:+5V #PWR0109
-U 1 1 6144619B
-P 2750 1650
-F 0 "#PWR0109" H 2750 1500 50  0001 C CNN
-F 1 "+5V" H 2765 1823 50  0000 C CNN
-F 2 "" H 2750 1650 50  0001 C CNN
-F 3 "" H 2750 1650 50  0001 C CNN
-	1    2750 1650
-	1    0    0    -1
-$EndComp
-$Comp
-L power:+5V #PWR0110
-U 1 1 614466A8
-P 3900 1650
-F 0 "#PWR0110" H 3900 1500 50  0001 C CNN
-F 1 "+5V" H 3915 1823 50  0000 C CNN
-F 2 "" H 3900 1650 50  0001 C CNN
-F 3 "" H 3900 1650 50  0001 C CNN
-	1    3900 1650
-	1    0    0    -1
-$EndComp
-$Comp
-L power:+5V #PWR0111
-U 1 1 6144723B
-P 5050 1650
-F 0 "#PWR0111" H 5050 1500 50  0001 C CNN
-F 1 "+5V" H 5065 1823 50  0000 C CNN
-F 2 "" H 5050 1650 50  0001 C CNN
-F 3 "" H 5050 1650 50  0001 C CNN
-	1    5050 1650
-	1    0    0    -1
-$EndComp
-$Comp
-L power:+5V #PWR0112
-U 1 1 614479FF
-P 5050 2800
-F 0 "#PWR0112" H 5050 2650 50  0001 C CNN
-F 1 "+5V" H 5065 2973 50  0000 C CNN
-F 2 "" H 5050 2800 50  0001 C CNN
-F 3 "" H 5050 2800 50  0001 C CNN
-	1    5050 2800
-	1    0    0    -1
-$EndComp
-$Comp
-L power:+5V #PWR0114
-U 1 1 61448221
-P 3900 2800
-F 0 "#PWR0114" H 3900 2650 50  0001 C CNN
-F 1 "+5V" H 3915 2973 50  0000 C CNN
-F 2 "" H 3900 2800 50  0001 C CNN
-F 3 "" H 3900 2800 50  0001 C CNN
-	1    3900 2800
-	1    0    0    -1
-$EndComp
-$Comp
-L power:+5V #PWR0115
-U 1 1 61448C3E
-P 2750 2800
-F 0 "#PWR0115" H 2750 2650 50  0001 C CNN
-F 1 "+5V" H 2765 2973 50  0000 C CNN
-F 2 "" H 2750 2800 50  0001 C CNN
-F 3 "" H 2750 2800 50  0001 C CNN
-	1    2750 2800
-	1    0    0    -1
-$EndComp
 Wire Wire Line
 	5500 1950 5500 2550
@@
 	1100 4200 1100 4250
 Wire Wire Line
-	1500 4250 1500 4350
-Wire Wire Line
 	1500 4250 1900 4250
 Wire Wire Line
@@
 Wire Wire Line
 	1500 4200 1500 4250
-$Comp
-L power:GND #PWR0123
-U 1 1 61442949
-P 1500 4350
-F 0 "#PWR0123" H 1500 4100 50  0001 C CNN
-F 1 "GND" H 1505 4177 50  0000 C CNN
-F 2 "" H 1500 4350 50  0001 C CNN
-F 3 "" H 1500 4350 50  0001 C CNN
-	1    1500 4350
-	1    0    0    -1
-$EndComp
 Connection ~ 1500 3800
 Wire Wire Line
@@
 Wire Wire Line
 	700  3900 700  3800
-$Comp
-L power:+5V #PWR0122
-U 1 1 614416E4
-P 1500 3700
-F 0 "#PWR0122" H 1500 3550 50  0001 C CNN
-F 1 "+5V" H 1515 3873 50  0000 C CNN
-F 2 "" H 1500 3700 50  0001 C CNN
-F 3 "" H 1500 3700 50  0001 C CNN
-	1    1500 3700
-	1    0    0    -1
-$EndComp
 $Comp
 L Device:C C1
@@
 	3750 5200 4150 5200
 NoConn ~ 3750 4800
+$Comp
+L Connector:AudioJack4 J1
+U 1 1 61864C23
+P 2550 6700
+F 0 "J1" H 2507 7025 50  0000 C CNN
+F 1 "AudioJack4" H 2507 6934 50  0000 C CNN
+F 2 "Random-keyboard-parts:PJ-3200B-4A" H 2550 6700 50  0001 C CNN
+F 3 "~" H 2550 6700 50  0001 C CNN
+	1    2550 6700
+	1    0    0    -1
+$EndComp
+$Comp
+L power:GND #PWR0104
+U 1 1 6186601A
+P 2850 7000
+F 0 "#PWR0104" H 2850 6750 50  0001 C CNN
+F 1 "GND" H 2855 6827 50  0000 C CNN
+F 2 "" H 2850 7000 50  0001 C CNN
+F 3 "" H 2850 7000 50  0001 C CNN
+	1    2850 7000
+	1    0    0    -1
+$EndComp
+Wire Wire Line
+	2750 6900 2850 6900
+Wire Wire Line
+	2850 6900 2850 7000
+Text Label 3850 6650 2    50   ~ 0
+DATA
+Wire Wire Line
+	2750 6600 2850 6600
+Wire Wire Line
+	2850 6600 2850 6500
+Wire Wire Line
+	2750 6700 3050 6700
+Text Label 4150 6400 2    50   ~ 0
+SDA
+Wire Wire Line
+	3050 6800 2750 6800
+Text Label 3850 7150 2    50   ~ 0
+SCL
+$Comp
+L Device:Jumper JP2
+U 1 1 618B0547
+P 3650 6400
+F 0 "JP2" H 3650 6175 50  0000 C CNN
+F 1 "SDA Jumper" H 3650 6266 50  0000 C CNN
+F 2 "Jumper:SolderJumper-2_P1.3mm_Open_Pad1.0x1.5mm" H 3650 6400 50  0001 C CNN
+F 3 "~" H 3650 6400 50  0001 C CNN
+	1    3650 6400
+	-1   0    0    1
+$EndComp
+Wire Wire Line
+	3950 6400 4150 6400
+Wire Wire Line
+	3350 6400 3050 6400
+Wire Wire Line
+	3050 6400 3050 6700
+$Comp
+L Jumper:Jumper_3_Open JP1
+U 1 1 618F5015
+P 3500 6900
+F 0 "JP1" V 3454 6986 50  0000 L CNN
+F 1 "Serial/SCL Jumper" V 3545 6986 50  0000 L CNN
+F 2 "Jumper:SolderJumper-3_P1.3mm_Open_Pad1.0x1.5mm" H 3500 6900 50  0001 C CNN
+F 3 "~" H 3500 6900 50  0001 C CNN
+	1    3500 6900
+	0    1    1    0
+$EndComp
+Wire Wire Line
+	3500 6650 3850 6650
+Wire Wire Line
+	3500 7150 3850 7150
+Wire Wire Line
+	3050 6800 3050 6900
+Wire Wire Line
+	3050 6900 3350 6900
+NoConn ~ 2550 4800
+NoConn ~ 3750 5400
+Wire Wire Line
+	3750 5100 3800 5100
+Wire Wire Line
+	1950 5100 1950 5000
+Wire Wire Line
+	1950 5000 2450 5000
+Wire Wire Line
+	2550 5100 2450 5100
+Wire Wire Line
+	2450 5100 2450 5000
+Connection ~ 2450 5000
+Wire Wire Line
+	2450 5000 2550 5000
+NoConn ~ 5350 3100
+$Comp
+L power:VCC #PWR0102
+U 1 1 6199D020
+P 2850 6500
+F 0 "#PWR0102" H 2850 6350 50  0001 C CNN
+F 1 "VCC" H 2865 6673 50  0000 C CNN
+F 2 "" H 2850 6500 50  0001 C CNN
+F 3 "" H 2850 6500 50  0001 C CNN
+	1    2850 6500
+	1    0    0    -1
+$EndComp
+$Comp
+L power:VCC #PWR0107
+U 1 1 619B47FD
+P 3800 5100
+F 0 "#PWR0107" H 3800 4950 50  0001 C CNN
+F 1 "VCC" V 3815 5273 50  0000 C CNN
+F 2 "" H 3800 5100 50  0001 C CNN
+F 3 "" H 3800 5100 50  0001 C CNN
+	1    3800 5100
+	0    1    1    0
+$EndComp
+$Comp
+L power:VCC #PWR0109
+U 1 1 619C37F5
+P 1500 3700
+F 0 "#PWR0109" H 1500 3550 50  0001 C CNN
+F 1 "VCC" H 1515 3873 50  0000 C CNN
+F 2 "" H 1500 3700 50  0001 C CNN
+F 3 "" H 1500 3700 50  0001 C CNN
+	1    1500 3700
+	1    0    0    -1
+$EndComp
+$Comp
+L power:VCC #PWR0110
+U 1 1 619D1F24
+P 2750 1650
+F 0 "#PWR0110" H 2750 1500 50  0001 C CNN
+F 1 "VCC" H 2765 1823 50  0000 C CNN
+F 2 "" H 2750 1650 50  0001 C CNN
+F 3 "" H 2750 1650 50  0001 C CNN
+	1    2750 1650
+	1    0    0    -1
+$EndComp
+$Comp
+L power:VCC #PWR0111
+U 1 1 619D9481
+P 3900 1650
+F 0 "#PWR0111" H 3900 1500 50  0001 C CNN
+F 1 "VCC" H 3915 1823 50  0000 C CNN
+F 2 "" H 3900 1650 50  0001 C CNN
+F 3 "" H 3900 1650 50  0001 C CNN
+	1    3900 1650
+	1    0    0    -1
+$EndComp
+$Comp
+L power:VCC #PWR0112
+U 1 1 619E085D
+P 5050 1650
+F 0 "#PWR0112" H 5050 1500 50  0001 C CNN
+F 1 "VCC" H 5065 1823 50  0000 C CNN
+F 2 "" H 5050 1650 50  0001 C CNN
+F 3 "" H 5050 1650 50  0001 C CNN
+	1    5050 1650
+	1    0    0    -1
+$EndComp
+$Comp
+L power:VCC #PWR0114
+U 1 1 619F696E
+P 3900 2800
+F 0 "#PWR0114" H 3900 2650 50  0001 C CNN
+F 1 "VCC" H 3915 2973 50  0000 C CNN
+F 2 "" H 3900 2800 50  0001 C CNN
+F 3 "" H 3900 2800 50  0001 C CNN
+	1    3900 2800
+	1    0    0    -1
+$EndComp
+$Comp
+L power:VCC #PWR0115
+U 1 1 619FDEFB
+P 5050 2800
+F 0 "#PWR0115" H 5050 2650 50  0001 C CNN
+F 1 "VCC" H 5065 2973 50  0000 C CNN
+F 2 "" H 5050 2800 50  0001 C CNN
+F 3 "" H 5050 2800 50  0001 C CNN
+	1    5050 2800
+	1    0    0    -1
+$EndComp
+$Comp
+L power:VCC #PWR0122
+U 1 1 61A0D396
+P 5400 4500
+F 0 "#PWR0122" H 5400 4350 50  0001 C CNN
+F 1 "VCC" V 5415 4673 50  0000 C CNN
+F 2 "" H 5400 4500 50  0001 C CNN
+F 3 "" H 5400 4500 50  0001 C CNN
+	1    5400 4500
+	0    1    1    0
+$EndComp
+$Comp
+L power:GND #PWR0113
+U 1 1 61A1C14C
+P 1500 4350
+F 0 "#PWR0113" H 1500 4100 50  0001 C CNN
+F 1 "GND" H 1505 4177 50  0000 C CNN
+F 2 "" H 1500 4350 50  0001 C CNN
+F 3 "" H 1500 4350 50  0001 C CNN
+	1    1500 4350
+	1    0    0    -1
+$EndComp
+Wire Wire Line
+	1500 4350 1500 4250
+$Comp
+L power:VCC #PWR0123
+U 1 1 61861826
+P 2750 2800
+F 0 "#PWR0123" H 2750 2650 50  0001 C CNN
+F 1 "VCC" H 2765 2973 50  0000 C CNN
+F 2 "" H 2750 2800 50  0001 C CNN
+F 3 "" H 2750 2800 50  0001 C CNN
+	1    2750 2800
+	1    0    0    -1
+$EndComp
 $EndSCHEMATC

Commit message: WIP v2
Connections:
- net ENC_A: now also U1.20 (PF4); no longer U1.19 (PF5)
- net ENC_B: now also U1.19 (PF5); no longer U1.20 (PF4)
Changed lines of the file:
@@
 ROW_0
 Text Label 4150 5300 2    50   ~ 0
-ENC_A
+ENC_B
 Text Label 8700 5750 0    50   ~ 0
 COL_0
@@
 	2150 5900 2550 5900
 Text Label 4150 5200 2    50   ~ 0
-ENC_B
+ENC_A
 Wire Wire Line
 	3750 5200 4150 5200
